Commit message: feat: Slam_map_toolbox
- Criação de um mapa slam
- Uso do ACLM

File: src/description/robot.urdf.xacro (robot description, xacro)
@@ -4,5 +4,5 @@
     <xacro:include filename="gazebo_control.xacro"/>
     <xacro:include filename="lidar.xacro"/>
-    <!--<xacro:include filename="camera.xacro"/>-->
-    <xacro:include filename="camera_depth.xacro"/>
+    <xacro:include filename="camera.xacro"/>
+    <!--<xacro:include filename="camera_depth.xacro"/>-->
 </robot>

File: src/description/robot_core.xacro (robot description, xacro)
@@ -19,4 +19,12 @@
     <!-- Base link -->
     <link name="base_link">
+    </link>
+    <!-- BASE_FOOTPRINT LINK -->
+    <joint name="base_footprint_joint" type="fixed">
+        <parent link="base_link"/>
+        <child link="base_footprint"/>
+        <origin xyz="0 0 0" rpy="0 0 0"/>
+    </joint>
+    <link name="base_footprint">
     </link>
     <!-- Chassis link -->
